Commit message: fixed issues with world/ and the urdf files to get gazebo launching

File: description/robot.urdf.xacro (robot description, xacro)
@@ -1,5 +1,5 @@
 <?xml version="1.0"?>
 <robot xmlns:xacro="http://www.ros.org/wiki/xacro"  name="robot">
-    <xacro:include filename="inertial_macros.xacro"/>
-    <xacro:include filename="robot_core.xacro"/>
+    <xacro:include filename="$(find articubot_one)/description/inertial_macros.xacro"/>
+    <xacro:include filename="$(find articubot_one)/description/robot_core.xacro"/>
 </robot>

File: description/robot_core.xacro (robot description, xacro)
@@ -20,99 +20,98 @@
     <!-- Essentially, a joint is the initial declaration (focused on relationship to other joints)
         and the link is the finer details such as visuals, geometry, material, and reference point (origin) -->
-    <!-- Start of base_link -->
-    <link name="base_link">
-        <!-- CHASSIS -->
-        <joint name="chassis_joint" type="fixed">
-            <parent link="base_link"/>
-            <child link="chassis"/>
-            <origin xyz="-0.1 0 0"/>
-        </joint>
-        <link name="chassis">
-            <visual>
-                <origin xyz="0.15 0 0 0.075" rpy="0 0 0"/>
-                <geometry>
-                    <box size="0.3 0.3 0.15"/>
-                </geometry>
-                <material name="white"/>
-            </visual>
-            <collision>
-                <origin xyz="0.15 0 0 0.075" rpy="0 0 0"/>
-                <geometry>
-                    <box size="0.3 0.3 0.15"/>
-                </geometry>
-            </collision>
-            <xacro:inertial_box mass="0.5" x="0.3" y="0.3" z="0.15">
-                <origin xyz="0.15 0 0.075" rpy="0 0 0"/>
-            </xacro:inertial_box>
-        </link>
-        <!-- LEFT WHEEL -->
-        <joint name="left_wheel_joint" type="continuous">
-            <parent link="base_link"/>
-            <child link="left_wheel"/>
-            <origin xyz="0 0.175 0" rpy="-${pi/2} 0 0"/>
-            <axis xyz="0 0 1"/>
-        </joint>
-        <link name="left_wheel">
-            <visual>
-                <geometry>
-                    <cylinder radius="${wheel_radius}" length="${wheel_length}"/>
-                </geometry>
-                <material name="blue"/>
-            </visual>
-            <collision>
-                <geometry>
-                    <cylinder radius="${wheel_radius}" length="${wheel_length}"/>
-                </geometry>
-            </collision>
-            <xacro:inertial_cylinder mass="0.1" length="${wheel_length}" radius="${wheel_radius}">
-                <origin xyz="0 0 0" rpy="0 0 0"/>
-            </xacro:inertial_cylinder>
-        </link>
-        <!-- RIGHT WHEEL -->
-        <joint name="right_wheel_joint" type="continuous">
-            <parent link="base_link"/>
-            <child link="right_wheel"/>
-            <origin xyz="0 -0.175 0" rpy="${pi/2} 0 0"/>
-            <axis xyz="0 0 -1"/>
-        </joint>
-        <link name="right_wheel">
-            <visual>
-                <geometry>
-                    <cylinder radius="${wheel_radius}" length="${wheel_length}"/>
-                </geometry>
-                <material name="blue"/>
-            </visual>
-            <collision>
-                <geometry>
-                    <cylinder radius="${wheel_radius}" length="${wheel_length}"/>
-                </geometry>
-            </collision>
-            <xacro:inertial_cylinder mass="0.1" length="${wheel_length}" radius="${wheel_radius}">
-                <origin xyz="0 0 0" rpy="0 0 0"/>
-            </xacro:inertial_cylinder>
-        </link>
-        <!-- CASTER WHEEL -->
-        <joint name="caster_wheel_joint" type="fixed">
-            <parent link="chassis"/>
-            <child link="caster_wheel"/>
-            <origin xyz="0.24 0.0 0.0" rpy="0.0 0.0 0.0"/>
-        </joint>
-        <link name="caster_wheel">
-            <visual>
-                <geometry>
-                    <sphere radius="${caster_wheel_radius}"/>
-                </geometry>
-                <material name="black"/>
-            </visual>
-            <collision>
-                <geometry>
-                    <sphere radius="${caster_wheel_radius}"/>
-                </geometry>
-            </collision>
-            <xacro:inertial_sphere mass="0.1" radius="${caster_wheel_radius}">
-                <<origin xyz="0 0 0" rpy="0 0 0"/>
-            </xacro:inertial_sphere>
-        </link>
-    <!-- End of base_link -->
+    <!-- BASE LINK -->
+    <link name="base_link"></link>
+    <!-- CHASSIS -->
+    <joint name="chassis_joint" type="fixed">
+        <parent link="base_link"/>
+        <child link="chassis"/>
+        <origin xyz="-0.1 0 0"/> <!-- The joint origin defines the pose (position + orientation)
+                                      of the child link relative to the parental link. These are offsets not coordinates -->
+    </joint>
+    <link name="chassis">
+        <visual>
+            <origin xyz="0.15 0 0.075" rpy="0 0 0"/> <!-- the pose of the geometry inside the link's own coordinate frame -->
+            <geometry>
+                <box size="0.3 0.3 0.15"/>
+            </geometry>
+            <material name="white"/>
+        </visual>
+        <collision>
+            <origin xyz="0.15 0 0.075" rpy="0 0 0"/>
+            <geometry>
+                <box size="0.3 0.3 0.15"/>
+            </geometry>
+        </collision>
+        <xacro:inertial_box mass="0.5" x="0.3" y="0.3" z="0.15">
+            <origin xyz="0.15 0 0.075" rpy="0 0 0"/>
+        </xacro:inertial_box>
+    </link>
+    <!-- LEFT WHEEL -->
+    <joint name="left_wheel_joint" type="continuous">
+        <parent link="base_link"/>
+        <child link="left_wheel"/>
+        <origin xyz="0 0.175 0" rpy="-${pi/2} 0 0"/>
+        <axis xyz="0 0 1"/>
+    </joint>
+    <link name="left_wheel">
+        <visual>
+            <geometry>
+                <cylinder radius="${wheel_radius}" length="${wheel_length}"/>
+            </geometry>
+            <material name="blue"/>
+        </visual>
+        <collision>
+            <geometry>
+                <cylinder radius="${wheel_radius}" length="${wheel_length}"/>
+            </geometry>
+        </collision>
+        <xacro:inertial_cylinder mass="0.1" length="${wheel_length}" radius="${wheel_radius}">
+            <origin xyz="0 0 0" rpy="0 0 0"/>
+        </xacro:inertial_cylinder>
+    </link>
+    <!-- RIGHT WHEEL -->
+    <joint name="right_wheel_joint" type="continuous">
+        <parent link="base_link"/>
+        <child link="right_wheel"/>
+        <origin xyz="0 -0.175 0" rpy="${pi/2} 0 0"/>
+        <axis xyz="0 0 -1"/>
+    </joint>
+    <link name="right_wheel">
+        <visual>
+            <geometry>
+                <cylinder radius="${wheel_radius}" length="${wheel_length}"/>
+            </geometry>
+            <material name="blue"/>
+        </visual>
+        <collision>
+            <geometry>
+                <cylinder radius="${wheel_radius}" length="${wheel_length}"/>
+            </geometry>
+        </collision>
+        <xacro:inertial_cylinder mass="0.1" length="${wheel_length}" radius="${wheel_radius}">
+            <origin xyz="0 0 0" rpy="0 0 0"/>
+        </xacro:inertial_cylinder>
+    </link>
+    <!-- CASTER WHEEL -->
+    <joint name="caster_wheel_joint" type="fixed">
+        <parent link="chassis"/>
+        <child link="caster_wheel"/>
+        <origin xyz="0.24 0.0 0.0" rpy="0.0 0.0 0.0"/>
+    </joint>
+    <link name="caster_wheel">
+        <visual>
+            <geometry>
+                <sphere radius="${caster_wheel_radius}"/>
+            </geometry>
+            <material name="black"/>
+        </visual>
+        <collision>
+            <geometry>
+                <sphere radius="${caster_wheel_radius}"/>
+            </geometry>
+        </collision>
+        <xacro:inertial_sphere mass="0.1" radius="${caster_wheel_radius}">
+            <origin xyz="0 0 0" rpy="0 0 0"/>
+        </xacro:inertial_sphere>
     </link>
 </robot>

Commit message: Keyboard control with gazebo working

File: description/robot.urdf.xacro (robot description, xacro)
@@ -1,5 +1,6 @@
 <?xml version="1.0"?>
 <robot xmlns:xacro="http://www.ros.org/wiki/xacro"  name="robot">
-    <xacro:include filename="$(find articubot_one)/description/inertial_macros.xacro"/>
-    <xacro:include filename="$(find articubot_one)/description/robot_core.xacro"/>
+    <xacro:include filename="inertial_macros.xacro"/>
+    <xacro:include filename="robot_core.xacro"/>
+    <xacro:include filename="gazebo_control.xacro"/>
 </robot>

File: description/robot_core.xacro (robot description, xacro)
@@ -14,5 +14,6 @@
         <color rgba="0 0 0 1"/>
     </material>
-    <!-- PROPERTIES (it would be good to add more to RE-RASSOR) -->
+    <!-- PROPERTIES
+    it would be good to add more to RE-RASSOR. Anywhere things are repeated should be a property -->
     <xacro:property name="wheel_radius" value="0.04"/>
     <xacro:property name="wheel_length" value="0.05"/>
@@ -47,4 +48,7 @@
         </xacro:inertial_box>
     </link>
+    <gazebo reference="chassis">
+        <material>Gazebo/White</material>
+    </gazebo>
     <!-- LEFT WHEEL -->
     <joint name="left_wheel_joint" type="continuous">
@@ -70,4 +74,7 @@
         </xacro:inertial_cylinder>
     </link>
+    <gazebo reference="left_wheel">
+        <material>Gazebo/Blue</material>
+    </gazebo>
     <!-- RIGHT WHEEL -->
     <joint name="right_wheel_joint" type="continuous">
@@ -93,4 +100,7 @@
         </xacro:inertial_cylinder>
     </link>
+    <gazebo reference="left_wheel">
+        <material>Gazebo/Blue</material>
+    </gazebo>
     <!-- CASTER WHEEL -->
     <joint name="caster_wheel_joint" type="fixed">
@@ -115,3 +125,8 @@
         </xacro:inertial_sphere>
     </link>
+    <gazebo reference="caster_wheel">
+        <material>Gazebo/Black</material>
+        <mu1 value="0.001"/>
+        <mu2 value="0.001"/>
+    </gazebo>
 </robot>

Commit message: added lidar. ran into issues using wsl. need to switch to linux

File: description/robot.urdf.xacro (robot description, xacro)
@@ -4,3 +4,4 @@
     <xacro:include filename="robot_core.xacro"/>
     <xacro:include filename="gazebo_control.xacro"/>
+    <xacro:include filename="lidar.xacro"/>
 </robot>

File: description/robot_core.xacro (robot description, xacro)
@@ -14,4 +14,7 @@
         <color rgba="0 0 0 1"/>
     </material>
+    <material name="red">
+        <color rgba="1 0 0 1"/>
+    </material>
     <!-- PROPERTIES
     it would be good to add more to RE-RASSOR. Anywhere things are repeated should be a property -->
@@ -21,5 +24,5 @@
     <!-- Essentially, a joint is the initial declaration (focused on relationship to other joints)
         and the link is the finer details such as visuals, geometry, material, and reference point (origin) -->
-    <!-- BASE LINK -->
+    <!-- BASES -->
     <link name="base_link"></link>
     <!-- CHASSIS -->
