Commit message: added limits to left and right wheel joint

File: src/articubot_one/description/robot_core.xacro (robot description, xacro)
@@ -60,4 +60,5 @@
         <origin xyz="0 0.175 0" rpy="-${pi/2} 0 0"/>
         <axis xyz="0 0 1"/>
+        <limit  effort="5" velocity="20"/>
     </joint>
     <link name="left_wheel">
@@ -86,4 +87,5 @@
         <origin xyz="0 -0.175 0" rpy="${pi/2} 0 0"/>
         <axis xyz="0 0 -1"/>
+        <limit  effort="5" velocity="20"/>
     </joint>
     <link name="right_wheel">
